File: circuit/circuit.sch (KiCad schematic (older format))
At the start: 7 parts, among them Q1 2N3904, U1 TL431LP

Commit message: edit schematic
Parts:
- R1: value 1k -> 3k3
Changed lines of the file:
@@
 P 4000 3000
 F 0 "R1" H 4070 3046 50  0000 L CNN
-F 1 "1k" H 4070 2955 50  0000 L CNN
+F 1 "3k3" H 4070 2955 50  0000 L CNN
 F 2 "" V 3930 3000 50  0001 C CNN
 F 3 "~" H 4000 3000 50  0001 C CNN
